Commit message: 3d: cradle bolts into heat-set inserts, camera mount hangs on the pedestal's front bolts
The cradle's four M3 nuts sat in a side channel "toward the centreline" - into the rail
box, which is solid there. A sealed cavity; every static check passed it, the first print
found it. A pocket open to the servo bore instead hollows the boss and puts land3g at the
strap's edge (--orient SF 1.33 → 0.77); bolts at |z| = 7 recover it (2.06) but move the
tray's seats, and a tray is printed. So: bolts stay at ±10.5, the boss stays solid, and
the screws land in M3 heat-set inserts (⌀5 × 6, hole INS_D 4.4, verify) pressed from the
flange side through the register spigot to a 1 mm lip in the boss. Screws M3 × 10.
cradle_insert_clear() sweeps the bore from open air, checks the lip and the tip.

The camera mount's two M3 went into nuts in the cradle's flange rib at y = 23 / 29: a
⌀3.4 hole through a rib 4 mm deep, and the rib was cut in two at both. Nothing else on the
mount can seat a head (1.3 mm skirt round the insertion path), so it has no screws now:
two tabs reach over the deck into pockets in the LiDAR base disc's underside and are
clamped by the pedestal's own front deck bolts. cam_tab() makes the tab and the pocket.
Key pocket gone from the tray and the cradle. A stop fin for the board was tried and
dropped.

Ladder: no !!, probes unchanged, cradle_front --orient 1.33 → 1.42, export --check upright
2.495 kg, flat trot 524.8. Also carries the other session's rear-panel change in
mini_dog.py (XT60 and balance lead off the panel, POWER.md) - same working tree.

Co-Authored-By: Claude Opus 5 (1M context) <noreply@anthropic.com>

File: ros2/smalldog_description/urdf/smalldog.urdf (robot description, URDF)
Before this commit: robot smalldog, 17 links, 16 joints
Links:
- link base_link: mass 1.55900 -> 1.56048
