Commit message: ros2: regenerate the description — sensors, terrain scene, honest masses
generate_model.py now carries the camera, the L2 and the GPS through camera.py
and lidar.py, writes the L2's parameters into robot.xml as <custom> numerics for
the C++ node to read back out of the compiled model, and emits scene_terrain.xml
plus meshes/terrain.png next to the flat scene. Foot sites grow to the real foot
radius, and the accelerometer is renamed imu_accel so mujoco_ros2_control's
<prefix>_quat/_gyro/_accel lookup finds it.

Masses follow the CAD's own fill factors and payload block instead of a local
copy: the robot is 2.496 kg, not 2.098 kg, and the difference is mostly infill
that was never modelled plus the camera, the GPS and the mast that carries it.

Generated output — `smalldog_description/scripts/generate_model.py` wrote every
file here, and it is the only thing that may.

Co-Authored-By: Claude Opus 5 (1M context) <noreply@anthropic.com>

File: ros2/smalldog_description/urdf/smalldog.urdf (robot description, URDF)
Before this commit: robot smalldog, 13 links, 12 joints
Links:
- added link camera_link
- added link camera_optical_frame
- added link gps_link
- added link lidar_link
- link base_link: mass 1.36252 -> 1.55920
- link fl_hip: mass 0.07642 -> 0.09039
- link fl_shin: mass 0.02741 -> 0.04659
- link fl_thigh: mass 0.08003 -> 0.09732
- link fr_hip: mass 0.07642 -> 0.09039
- link fr_shin: mass 0.02741 -> 0.04659
- link fr_thigh: mass 0.08003 -> 0.09732
- link rl_hip: mass 0.07642 -> 0.09039
- link rl_shin: mass 0.02741 -> 0.04659
- link rl_thigh: mass 0.08003 -> 0.09732
- link rr_hip: mass 0.07642 -> 0.09039
- link rr_shin: mass 0.02741 -> 0.04659
- link rr_thigh: mass 0.08003 -> 0.09732
Joints:
- added joint camera_joint: type fixed, parent base_link, child camera_link, origin xyz=0.0787343 0 0.0257543 rpy=0 -0.10472 0
- added joint camera_optical_joint: type fixed, parent camera_link, child camera_optical_frame, origin xyz=0 0 0 rpy=-1.5708 0 -1.5708
- added joint gps_joint: type fixed, parent base_link, child gps_link, origin xyz=-0.05200 0.00000 0.07260 rpy=0 0 0
- added joint lidar_link_joint: type fixed, parent base_link, child lidar_link, origin xyz=0.0734663 0 0.0914663 rpy=0 0.785398 0

Commit message: Put the thigh's cable-tie slots back to sharp rectangles
Rounding them was the obvious "corners concentrate stress" move, and measured
it buys nothing: thigh_A stall at 1.2 mm reads 23.19 MPa sharp, 23.15 obround,
22.95 obround stopping short of the pocket wall, 22.98 with no slot at all.
The slot is worth 0.2 MPa of 23.  The 2.0 mm arm spreads 15.7..18.5 over the
same four, which is one mesh's luck on an unconverged corner and must not be
read as a result either way.

The peak is somewhere else entirely: the knee sleeve's cable window leaves this
beam's two +-y walls unsupported over the 15 mm it spans, and both hot cells
sit 0.3 mm inside its edges.  Bounding that window in local z is the change
that would move the number, and it touches all three sleeves, so it is its own
job.  The comment in thigh() carries the numbers.

Simpler geometry, and 0.1 g lighter: 2.4964 -> 2.4963 kg.  The ROS 2
description is regenerated from it in the same commit.

Co-Authored-By: Claude Opus 5 (1M context) <noreply@anthropic.com>

File: ros2/smalldog_description/urdf/smalldog.urdf (robot description, URDF)
Before this commit: robot smalldog, 17 links, 16 joints
Links:
- link fl_thigh: mass 0.09732 -> 0.09731
- link fr_thigh: mass 0.09732 -> 0.09731
- link rl_thigh: mass 0.09732 -> 0.09731
- link rr_thigh: mass 0.09732 -> 0.09731

Commit message: sim: the ROS 2 model gets the servo the CAD actually specifies
generate_model.py kept J_EFF = 3.0 and J_VEL = 4.7, rounded copies of
mini_dog's SERVO_STALL_NM = 2.94 and SERVO_NOLOAD_RADS = 4.71.  Both now
read from the source, which closes the third and last of these.

This one was worse than "a constant written twice", and the sharper
statement is worth having: export_sim.py has read both numbers all along,
so out/sim/mini_dog.xml has said forcerange="-2.94 2.94" and effort="2.94"
this whole time while the ROS 2 model said 3.0.  The two exporters were
not duplicating a constant, they were emitting robots with different servo
strength, and which sim you loaded decided how strong the servo was.  rl/
loads the ROS 2 one, so that was the one that mattered.

RE-BASELINED, control first on the unchanged model, same machine, same seeds:

  flat trot        781.4 -> 781.6 mm        (+0.2 mm, deterministic both sides)
  terrain s7..s12  622 +-27 -> 618 +-37 mm  (-5 mm of means against ~32 mm sd)
  course           4/7 both; reach 2512 -> 2606 mm, upright both

I deferred this fix two commits ago on the grounds that -2 % of servo
torque could move the operating point, since 11 g of mass moves that same
trot 778 -> 597 mm.  That was wrong, and the negative result is the more
useful half of this commit: 2 % of torque is a much larger relative
perturbation than 4 permille of mass and it moved the trot 0.2 mm.  The
bifurcation is under the mass axis; the torque axis is flat.  CLAUDE.md
now says that explicitly, because the old wording implied the gait was
fragile to everything and that is what held a harmless change.

Two other corrections to CLAUDE.md's step 6, both found by running the
control rather than trusting the file:

  - the recorded course baselines (5/7 at 2790/2883/2896 mm) do not
    reproduce on the current tree.  The UNCHANGED model reads 4/7 and
    2512 mm at 2.496 kg, against 2.499 kg recorded.  They are now marked
    as history rather than as a target, with an instruction to re-baseline
    instead of chasing them.
  - the terrain sweep pair is recorded as a pair, because a single seed
    cannot distinguish 622 +-27 from 618 +-37 and the file should not
    invite anyone to try.

mini_dog.py is untouched, so no rebuild and no FEA: geometry, masses and
joint limits are bit-identical and the only diff in the description is
forcerange, twelve effort/velocity pairs, and joint_velocity_limit.

Co-Authored-By: Claude Opus 5 <noreply@anthropic.com>

File: ros2/smalldog_description/urdf/smalldog.urdf (robot description, URDF)
Before this commit: robot smalldog, 17 links, 16 joints
Joints:
- joint fl_knee: limit lower=-1.8500 upper=1.8500 effort=3.0 velocity=4.7 -> lower=-1.8500 upper=1.8500 effort=2.94 velocity=4.71
- joint fl_pitch: limit lower=-1.3000 upper=1.3000 effort=3.0 velocity=4.7 -> lower=-1.3000 upper=1.3000 effort=2.94 velocity=4.71
- joint fl_roll: limit lower=-0.9000 upper=0.9000 effort=3.0 velocity=4.7 -> lower=-0.9000 upper=0.9000 effort=2.94 velocity=4.71
- joint fr_knee: limit lower=-1.8500 upper=1.8500 effort=3.0 velocity=4.7 -> lower=-1.8500 upper=1.8500 effort=2.94 velocity=4.71
- joint fr_pitch: limit lower=-1.3000 upper=1.3000 effort=3.0 velocity=4.7 -> lower=-1.3000 upper=1.3000 effort=2.94 velocity=4.71
- joint fr_roll: limit lower=-0.9000 upper=0.9000 effort=3.0 velocity=4.7 -> lower=-0.9000 upper=0.9000 effort=2.94 velocity=4.71
- joint rl_knee: limit lower=-1.8500 upper=1.8500 effort=3.0 velocity=4.7 -> lower=-1.8500 upper=1.8500 effort=2.94 velocity=4.71
- joint rl_pitch: limit lower=-1.3000 upper=1.3000 effort=3.0 velocity=4.7 -> lower=-1.3000 upper=1.3000 effort=2.94 velocity=4.71
- joint rl_roll: limit lower=-0.9000 upper=0.9000 effort=3.0 velocity=4.7 -> lower=-0.9000 upper=0.9000 effort=2.94 velocity=4.71
- joint rr_knee: limit lower=-1.8500 upper=1.8500 effort=3.0 velocity=4.7 -> lower=-1.8500 upper=1.8500 effort=2.94 velocity=4.71
- joint rr_pitch: limit lower=-1.3000 upper=1.3000 effort=3.0 velocity=4.7 -> lower=-1.3000 upper=1.3000 effort=2.94 velocity=4.71
- joint rr_roll: limit lower=-0.9000 upper=0.9000 effort=3.0 velocity=4.7 -> lower=-0.9000 upper=0.9000 effort=2.94 velocity=4.71

Commit message: cad: the foot bolt gets a hole that reaches the outside
foot() cut its M3 clearance hole from zf-6 and its head pocket from
zf-1, both written as if the dome's radius were 6 rather than
FOOT_D/2 = 13.  The hole therefore opened 7 mm INSIDE the solid and
never broke the sole at all, and the pocket's one annulus - at zf-1,
between r 1.7 and 3.4 - faced up, while the nut above pulls the bolt
up and the head needs a face looking down.  So step 4 of README's
assembly order was not merely awkward, it was impossible: there was
no path in and nothing to bear on.

The bolt was specified as M3 x 16.  The span from the sole to the
nut's far face is 28 mm, so no position of the head could ever have
reached - which is the tell that the number was never checked against
the solid.  Both cuts are now anchored to FOOT_D and start below the
sole, the pocket ceiling at FOOT_CB_Z is the bearing shoulder, and
the length follows from FOOT_CB_Z + FOOT_NUT_Z + M3_NUT_H rather than
sitting in the BOM as a free number.

None of the existing checks could see this: isValid() does not mind a
hole that goes nowhere, interference() only covers the static body
parts, and rom_scan only covers what moves.  foot_bolt_check() now
probes the real solid along the axis and build() prints a foot bolt:
line beside body clear: and gps clear:.

Only foot() changed shape - hip_bracket, thigh and shin are identical,
so only the four TPU feet are reprinted, and the bolt becomes M3 x 30.

Verified per CLAUDE.md, each arm against a control run of the
unchanged tree in a worktree at HEAD:
  fea.py --all      inter-layer SF unchanged at stall, 4.8 / 1.2 / 2.4
  export_sim --check  2.497 kg, 4 feet down, upright +1.00, base 187 mm
  ROS 2 mass        2.496 kg both; shin+foot link 0.04659 -> 0.04652 kg
  flat trot         781.6 -> 782.0 mm, same seed, deterministic
  terrain seeds 7-12  618 +-37 mm -> 642 +-59 mm, the same distribution
                    (the control reproduces the 618 +-37 in CLAUDE.md)
  course            4/7 at 2606 mm -> 5/7 at 2716 mm, inside its spread

The sole now meets the ground as a ring at zf-12.60 instead of a point
at zf-13, so the foot's print bbox is 24.6 mm rather than 25.0.  The
sim does not see it - the ROS 2 model merges the foot into the shin and
collides with a primitive.

Co-Authored-By: Claude Opus 5 (1M context) <noreply@anthropic.com>

File: ros2/smalldog_description/urdf/smalldog.urdf (robot description, URDF)
Before this commit: robot smalldog, 17 links, 16 joints
Links:
- link fl_shin: mass 0.04659 -> 0.04652
- link fr_shin: mass 0.04659 -> 0.04652
- link rl_shin: mass 0.04659 -> 0.04652
- link rr_shin: mass 0.04659 -> 0.04652

Commit message: cad: the IMU gets a mounting point, and both exporters read it
generate_model.py wrote <site name="imu" pos="0 0 0"> while export_sim.py
wrote BODY_Z1, so the two files described robots whose accelerometers sat
25 mm apart - the servo-mass / MJ_* / SERVO_STALL_NM defect a fourth time.
This one had been shipping into training: rl/ loads the ROS 2 model, so the
offset was in the observation the policy learns from.

What makes it different from the three before it is that nothing inside 3d/
could have caught it.  It took rl/checks/imu_placement.py, which adds real
accelerometers at candidate mounts through MjSpec and compares them against
the site the model ships.  Its number is the argument for the position, not
a warning to note: an accelerometer offset by r from the `imu` site reads
omega x (omega x r) + alpha x r on top of gravity, and on the existing
0.2 m/s trot that reaches 9.0 m/s2 - 42 deg of apparent tilt - for a board
out on the deck beside the Pi, against 25 deg on the centreline.  Once site
and board agree the term stops being an error at all; what remains is that
the swing the policy observes, and every residual mounting error with it,
scale with |r|.  Reproduced here on the mac before anything was moved.

So the board is placed, not just pointed at.  The bay decided the rest and
it is tight.  On the centreline the only opening is the deck's own window at
x +-16, |y| <= 34; the pack's top is at BODY_Z0+BATT_H = 21.4 and the deck's
underside at BODY_Z1 = 25.  That is 3.6 mm, of which the board and its
components are 2.8.  The deck's 4 mm above is not free either - it is
OPI_BOX's floor.  The board therefore bolts UP under two tabs bridging the
window, component face down, and the M2.5 nut sits in a channel that takes
exactly DECK_T - M25_NUT_H - NUT_CLR and comes out flush with the deck's top
face, so nothing reaches into the Pi's envelope.  0.80 mm of air is left
under the board and the build prints it every run; imu_clear() checks it,
because the pack is a payload and interference() cannot see one.

IMU_STACK = 1.2 is headerless and that is a build constraint, not a
tolerance: a 2.54 mm pin header is 8.5 mm and misses this bay by 3x.
ref/imu/README.md says so, and says the six wires get soldered to the pads.
Every number in that file is a transcription - no BMI088 has been measured -
so it is flagged **verify** throughout, like ref/camera/.  If the real board
is thicker, the 0.80 mm is where it shows, and the fix is in ref/imu/.

Verified, the whole ladder, against baselines taken on the unchanged tree
first (2.496 kg):

  build          all parts valid; body clear now includes the board itself;
                 imu clear +0.80 mm
  FEA --all      inter-layer SF unmoved - thigh_A stall 1.2, hip_bracket_A
                 2.4, shin_A 4.8.  Only in-plane shin_A stand2/stand4 moves,
                 58.9 -> 58.8, which is +3 g in the ground load cases.
  export_sim     4 feet down, upright +1.00; terrain the same; camera axis
                 (+0.99 0 +0.10); urdf and mjcf agree
  flat trot      782.0 -> 781.7 mm at 2.496 -> 2.499 kg
  course         5/7, 2692 -> 2878 mm
  terrain        642 +-59 -> 649 +-53 mm over seeds 7..12

The terrain arm is why the sweep is here rather than one number.  The
default seed alone read 574.9 -> 552.3, a 22.6 mm drop that looks like a
regression and is not: the means differ by 7 mm against a 55 mm spread and
the changed arm is nominally higher.  The control arm was run from a
detached worktree at 7f66997, same binary, same seeds.  CLAUDE.md already
says to read this arm over a sweep or not at all; this is what that costs
and it is cheap.

The flat trot is the one that was actually at risk - it is chaotic in mass
at this operating point, 11 g moves it 180 mm - and +3 g moved it 0.3 mm.

Co-Authored-By: Claude Opus 5 (1M context) <noreply@anthropic.com>

File: ros2/smalldog_description/urdf/smalldog.urdf (robot description, URDF)
Before this commit: robot smalldog, 17 links, 16 joints
Links:
- link base_link: mass 1.55920 -> 1.56250

Commit message: cad: the access bores inverted the chassis, and isValid() said it was fine
Working the MAC.md queue: five commits had changed 3d/ from a session with no
CadQuery, so none of it had been through a boolean.  Step 1 came back with
chassis_bottom at -0.3 cm3.

7e30e75 cut its four @6 bores BEFORE the rear connector pads were unioned on,
and the pads start at exactly the plane the bores end on - xw+WALL = -60.2
against the bores' BODY_L/2-WALL = 60.2.  They share no volume at all; the pad's
inner face was welded straight onto the bore's circular opening, and OCC's fuse
on that degenerate contact returned an INVERTED solid.  isValid() said True, so
nothing downstream noticed: 240 cm3 of chassis became a 2.5 x 14.9 x 6.9 mm
sliver, the ROM read hip_roll +0..+0, every interference() pair fired at once,
and the robot came out 280 g light.

Cut last, after everything that adds material near the path, and build() now
fails a part whose volume is not positive - the one-line check that names this
instead of five confusing ones.  Both are in 3d/CLAUDE.md now.

The rest of the ladder is green.  No inter-layer SF dropped anywhere;
hip_bracket_A improved (stand4 46.3 -> 46.7, land3g 7.7 -> 7.8) on the bigger
bearing area, thigh_A and shin_A identical.  ROM unmoved, no bbox moved,
export_sim --check stands it up 4 feet down upright +1.00, check_model 0 FAIL,
walk.py --dry-run 1050 ticks 0 late.

Mass is -4.15 g, not the -1.2 g MAC.md predicted: hub holes 1.3 g, access bores
2.9 g.  Control run beside it because that is inside the hypersensitive band -
flat 781.7 -> 782.4 mm, course 5/7 2892 -> 5/7 2893 mm, terrain over seeds 7..12
649 +-48 -> 625 +-89 mm.  Same distribution on all three.

NOT fixed, and now written up as the live item in MAC.md: the bores do not do
what they were cut to do.  The deck boss at (+-52, +-38) is full height and its
outer face is 2.4 mm inboard of the bore mouth, overlapping three of the four
screw axes by 5.05 and 2.05 mm - only y = 29 is reachable.  The outboard bore at
y = 43 reaches y = 46.00, the tray's OUTER skin, leaving 0.00 mm of wall at z=0.
An M3 head cannot pass that wall on that axis at all (45.75 vs 46.00).  And the
tilt budget is 12.5 deg, not the claimed 23.9 - the key pivots at the screw, at
the bore's far end, not at the bore's middle.  fork_access() prints "all six arms
break out" through all of it, because DRIVER_REACH = 7.5 against a 7.9 mm bore
keeps the probe inside the bore.  Fixing it is a design decision; three options
are in MAC.md.

Also in this commit, from a parallel session on this machine: bench_rig.py's
hub_bolts()/bolt_paths() - the same defect class, a hole cut before the union
that fills it back in, with the check that catches it.

Co-Authored-By: Claude Opus 5 (1M context) <noreply@anthropic.com>

File: ros2/smalldog_description/urdf/smalldog.urdf (robot description, URDF)
Before this commit: robot smalldog, 17 links, 16 joints
Links:
- link base_link: mass 1.56250 -> 1.55963
- link fl_hip: mass 0.09039 -> 0.09028
- link fl_shin: mass 0.04652 -> 0.04642
- link fl_thigh: mass 0.09731 -> 0.09720
- link fr_hip: mass 0.09039 -> 0.09028
- link fr_shin: mass 0.04652 -> 0.04642
- link fr_thigh: mass 0.09731 -> 0.09720
- link rl_hip: mass 0.09039 -> 0.09028
- link rl_shin: mass 0.04652 -> 0.04642
- link rl_thigh: mass 0.09731 -> 0.09720
- link rr_hip: mass 0.09039 -> 0.09028
- link rr_shin: mass 0.04652 -> 0.04642
- link rr_thigh: mass 0.09731 -> 0.09720

Commit message: cad: the hip's inboard fork screws are reached through the corner, and the leg turns
The four coaxial bores of 7e30e75 reached one screw of four (MAC.md, 2026-09-03):
a deck boss stood in front of two, the outboard one ran 0.2 mm inside the side wall,
and a coaxial bore only lets a key tilt 12 deg. No path into the tray can work - the
battery cradle's end stop closes every one within 18 mm.

Replaced by fork_access_channels(): two @6 channels per hip, on the "out" and "top"
positions of the hub circle, leaning KEY_TILT = 20 deg outboard, cut last on the
assembled chassis. In open air past the tray's front corner after 8 mm and 29 mm
(the second passes under the corner deck boss's screw hole and out through the side
vent). The screw circle turns with the leg, so two channels a quarter turn apart
serve all four screws - inboard arm first, leg turned by hand, deck and battery in
place. fork_channels_cover() checks the turn in closed form.

fork_access() now probes along the same lines for their whole 55 mm, i.e. to open
air, instead of stopping inside the bore; a failed boolean counts as blocked.

Ladder: all parts valid, ROM unchanged, FEA identical (nothing in the set touched),
export_sim --check upright, ROS 2 regenerated. Control beside it, same seeds:
flat 782.4 -> 781.8 mm, terrain seeds 7..12 625 +-95 -> 631 +-55 mm, course
5/7 2893 -> 4/7 2639 mm (the flip CLAUDE.md documents on the unchanged tree).
chassis_bottom 240.18 -> 239.8 cm3, total 2.495 kg either side.

A chassis already printed is a drill job, not a reprint - MAC.md, last section.

Co-Authored-By: Claude Fable 5.1 <noreply@anthropic.com>

File: ros2/smalldog_description/urdf/smalldog.urdf (robot description, URDF)
Before this commit: robot smalldog, 17 links, 16 joints
Links:
- link base_link: mass 1.55963 -> 1.55917

Commit message: cad: the hub screws are ISO 7380 button heads, and their heads were never in the model
The screws arrived: ISO 7380 M3 x 6, 2 mm hex socket. Two consequences.

The key for the hip channels is 2 mm, not 2.5 (KEY_D). And a button head is 1.65 mm
tall on an inboard arm that had 0.6 mm of air to the chassis gusset - the hip would
have bound on its own screw heads before it turned a degree, and no check saw it,
because like the thrust clamp's cap head the part in the way was hardware.

FORK_GAP 0.6 -> 1.1 (the gusset face moves back half a millimetre); the passive arm's
four holes get a FORK_CB = 1.2 counterbore; fork_screws() puts all eight heads on the
moving side of every rom_scan; head_clear() prints the head's air to the gusset and
the tip's distance to the servo case on every run: +0.65, +0.50 / +0.80 mm.

The counterbore also makes the passive screw an M3 x 6 - it was an M3 x 7, a length
nobody stocks - so the BOM is 96 x M3 x 6 and nothing else at the hubs.

Ladder against 89e5149: ROM with the heads swept unchanged; hip_bracket_A inter-layer
46.8 / 23.4 / 7.8 / 2.4 vs 46.7 / 23.3 / 7.8 / 2.4; export_sim upright, 2.493 kg;
ROS 2 regenerated (every hip/thigh/shin mesh - fork() is one part). Flat 781.8 ->
781.1 mm, terrain seeds 7..12 631 +-55 -> 657 +-35 mm, course 4/7 -> 3/7 at 2209 mm -
flagged in MAC.md as three chaotic samples on one seed, not acted on.

Co-Authored-By: Claude Fable 5.1 <noreply@anthropic.com>

File: ros2/smalldog_description/urdf/smalldog.urdf (robot description, URDF)
Before this commit: robot smalldog, 17 links, 16 joints
Links:
- link base_link: mass 1.55917 -> 1.55831
- link fl_hip: mass 0.09028 -> 0.09016
- link fl_shin: mass 0.04642 -> 0.04630
- link fl_thigh: mass 0.09720 -> 0.09707
- link fr_hip: mass 0.09028 -> 0.09016
- link fr_shin: mass 0.04642 -> 0.04630
- link fr_thigh: mass 0.09720 -> 0.09707
- link rl_hip: mass 0.09028 -> 0.09016
- link rl_shin: mass 0.04642 -> 0.04630
- link rl_thigh: mass 0.09720 -> 0.09707
- link rr_hip: mass 0.09028 -> 0.09016
- link rr_shin: mass 0.04642 -> 0.04630
- link rr_thigh: mass 0.09720 -> 0.09707
