Commit message: cad: the hip-roll cradles bolt on, and the rear panel opened into solid plastic
Carries TWO changes rather than one, and that is deliberate: they are interleaved in the
same files, and the generated ROS 2 description cannot be split between them without
leaving one commit's model stale against its own CAD - which 3d/CLAUDE.md forbids
outright.  Both ladders are in MAC.md.

1. THE BATTERY BECAME A MODULE (worked earlier the same day).  Six 21700 welded into a
   3 x 2 brick, heatshrunk, the BMS beside them, all of it in battery_case + battery_lid
   dropping into a seat recess as one payload.  The cradle's fins, end stops and front
   BMS bay are gone.  The binding constraint was height and it was not close, so the IMU
   moved out of the 3.6 mm over the pack and onto the deck's TOP face - which is a
   RE-BASELINE for rl/, not a defect: the site rose 7.6 mm and the observation moved with
   it (p95 0.60, max 4.28 m/s2, worst apparent tilt 23.6 deg).  A policy trained against
   the older model has to retrain, not fine-tune.

2. THE HIP-ROLL CRADLES ARE BOLTED PARTS.  cradle_front and cradle_rear, one off each,
   four M3 x 12 per end through a spigot register.  chassis_bottom goes from
   213 x 110 x 50 mm / 208 g to 126 x 92 x 50 / 127 g, so a tray change stops meaning
   "reprint four cradles and unbolt four servos", which is what was asked for.

   It started from a different report - that the cutouts on the back were blocked - and
   the two turned out to be one defect.  They WERE blocked, every one: the two rear
   cradles met across the centreline as a continuous 2.8 mm plate 1.2 mm behind the wall,
   and the XT mating halves stand proud to 0.3 mm INSIDE it.  Nothing could see it,
   because the cradles were chassis_bottom and a part cannot interfere with itself.  The
   flange is a frame now and the panel is laid out inside its opening; the XT60 did not
   fit there and moved above the cradle.

   The fork-access channels are deleted with it.  They existed because the roll joint's
   inboard arm faced the chassis and the fork could only go on after the cradle was welded
   to the tray; bolted, the fork goes on with the cradle in hand and all four screws are
   in open air (0 mm3 against the cradle, 569 against the cradle on the tray).  Eight @6
   holes out of the tray's corner posts and deck bosses, and fork_access() reads six arms
   instead of five.  An access problem that keeps needing cleverer holes was telling us
   the part boundary was in the wrong place.

   Three probes added, all of which caught something on their first run: panel_clear()
   (the blockage above), cradle_clear() (the ESP32 divider rib 0.5 mm into two screws'
   driver runs - its width was still derived from a BMS that moved weeks ago),
   cradle_head_clear() (eight screw heads 0.4 mm inside the battery pack; the part in the
   way is hardware, so nothing else could see it either).

   fea.py: cradle_front joins the set - a part carrying a whole leg through a bolted
   flange is what that script is for, and this geometry had never been analysed because
   it lived in chassis_bottom.  The first run found a 1.4 mm notch and a 27.6 mm step in
   the strap; peak 53.7 -> 29.7 MPa, deflection 1.58 -> 1.00 mm.  solve() gained a second
   traction patch so a stall torque on a bore CONCENTRIC with its own joint axis can be a
   couple instead of dividing by zero.

   It is still the weakest printed part on the robot: interlayer SF 1.35 at land3g on
   --orient, against 3.08 for thigh_A.  Not a regression - the version on the robot today
   is the notched one at 0.4, and it has not broken - but it is the number to watch, and
   the space that would fix it is swept by the fork over the +-90 deg roll ROM.

   MATERIALS in fea.py is now flagged UNVERIFIED, and that matters: its interlayer column
   is the in-plane column halved, one rule for four materials.  PA-CF looked like a free
   fix at 2.35 and is not - the fibres align with the extrusion and do nothing across the
   interface, the worst element here is 88 % tension ACROSS the layers, and break-even is
   s_z = 20, i.e. PA-CF must match PETG's layer adhesion just to draw.  Print PETG.

Gait, same seeds and same day, unchanged tree beside the changed one (2.493 -> 2.487 kg):
terrain seeds 7..12 498 +-81 -> 520 +-67 (one distribution, and it is the arm to read),
flat trot 595.2 -> 556.6 mm, course seeds 7/8/9 5-3-4 -> 1-5-4 obstacles, all upright
both sides.  An intermediate version 8 g lighter went DOWN on one course seed while its
terrain sweep was indistinguishable - read the course over seeds or not at all.

Co-Authored-By: Claude Opus 5 (1M context) <noreply@anthropic.com>

File: ros2/smalldog_description/urdf/smalldog.urdf (robot description, URDF)
Before this commit: robot smalldog, 17 links, 16 joints
Links:
- link base_link: mass 1.55831 -> 1.55324

Commit message: cad: the BMS is 60.13 x 37.2 x 5.9, and that cost the case its y retention
The last **verify** row on the battery module met the real board.  All three
catalogue numbers were wrong: 64 x 27 x 13 guessed against 60.13 x 37.2 x 5.9
measured, the thickness over the heatsink plate.  The orientation is forced by
the case - a 60.13 mm edge cannot stand up in a 43.6 mm interior.

The thickness is 7.1 mm under the guess and comes straight off BATT_IN_L, so
the module went 102.3 x 68.2 x 46.4 -> 95.2 x 68.1 x 46.4 and the robot lost
about 2 g.  BATT_X is deliberately not re-centred: holding it walks the heavy
brick 3.55 mm aft, the direction the module owed the CoM when the BMS went in
behind the cells.

What the measurement broke is not a fit, it is a claim.  battery_case's
docstring says the BMS is retained in all six directions with no fasteners,
and y was the case's own side walls closing on a 64.0 mm board.  The real one
leaves 2.4 mm a side - a loose PCB with wires on it inside a battery case.
BMS_SIDE_Y adds two ribs off the rear wall, floor to the board's top edge,
+1.2 g.

Ladder, with a control on the unchanged tree beside it: every part valid, ROM
unmoved, module clear 0.0/0.0 mm3 with the ribs in; not one FEA safety factor
moved; export_sim 2.486 kg, 187 mm, upright.  Gait - flat 481.4 vs 487.0 mm,
terrain seeds 7..12 350 +-31 vs 340 +-43 mm, course 2/7 1839, 2/7 1820,
2/7 1797 vs 2/7 1903, 2/7 1705, 0/7 1005, all upright.  The control came back
bit-for-bit on the fitted-actuator baseline in 3d/CLAUDE.md step 6, which is
what makes the after-numbers readable.

Still open on this part, and it is not a dimension: the board arrived with a
5S LiFePO4 sticker on it.  Check the 3S/4S jumpers and the charge cutoff on the
bench before the module is closed - those pads are unreachable behind a lid
whose two M2.5 are thread-forming.

Co-Authored-By: Claude Opus 5 (1M context) <noreply@anthropic.com>

File: ros2/smalldog_description/urdf/smalldog.urdf (robot description, URDF)
Before this commit: robot smalldog, 17 links, 16 joints
Links:
- link base_link: mass 1.55324 -> 1.55154

Commit message: cad: two printed combs hold the cells on a pitch, and the module grows by the gaps alone
`cell_holder`, x2, one at each end of the cells.  It exists because welding six
loose cylinders into a 3 x 2 brick by hand is the assembly step this design had
no answer for - the combs turn the six into one riggable object before any
nickel goes on.

The obvious holder is a frame round the outside of the array and it does not
fit: the module already has 1.4 mm to the deck and 0.5 mm to the deck screws'
nut bosses at |y| = 35.2.  So the caps are clipped flush with the outermost
cells' own tangent planes in both y and z - no material outboard of any cell
anywhere - and the module grows by the separator gaps alone, +0.8 in z and
+1.6 in y.  An 0.8 mm collar clipped at the tangent still leaves an 8.4 mm
flat, and a 21.3 mm cell does not leave through 8.4 mm.

`holder_clear()` probes both caps against the case and against all six cells,
because the cells are a payload and the holder lives inside another part's
cavity: neither `interference()` nor `isValid()` can see a cap drawn half a
millimetre too wide.  And `build()` now checks each part's SOLID COUNT against
`PART_SOLIDS` - the part came back as five loose pieces the first time, the two
clip planes meeting at each corner cell and orphaning a crescent of collar,
with `isValid()` and `Volume() > 0` both green.

The mass is +7 g and both exporters carry it off `md.cell_holders()`; the caps
are deliberately not in BODY_PARTS (invisible inside the case, no mesh wanted).

Step 6 re-baselined with a +7 g dead-mass control beside the unchanged tree,
because 7 g parked in ELECTRONICS_KG on unmoved geometry reproduces the same
picture the holder does - one terrain seed on its back, the course from 6/21 to
3/21 - so this is the documented mass cliff and not a geometry regression.
The flat trot was blind to all of it at 481/481/483 mm.

Co-Authored-By: Claude Opus 5 (1M context) <noreply@anthropic.com>

File: ros2/smalldog_description/urdf/smalldog.urdf (robot description, URDF)
Before this commit: robot smalldog, 17 links, 16 joints
Links:
- link base_link: mass 1.55154 -> 1.55858

Commit message: bench: the ST3215 makes 4.50 N*m, measured on a scale, not 2.94
PLAN.md step 2c, closed.  A printed C-frame with a 170 mm arm pressing an M6
anvil onto a 2 kg coffee scale, three duty rungs at 12 V: k_u = 0.400 N*m/V,
friction intercept -0.30 N*m, stall 4.50 N*m (4.38 read warm), residuals
+-0.05 N*m.

BOTH PREVIOUS ANSWERS WERE WRONG, IN OPPOSITE DIRECTIONS.  The register routes
implied 7.40 and the datasheet said 2.94; the truth is between them, so the
register channel is high by 1.64x - not the 2.2x the old note assumed - and the
datasheet is optimistic by 1.53x on top of that.  There was never one mis-scaling
to find.  The -0.30 N*m intercept is a third independent read on tau_c, against
the hysteresis ladder's 0.43.

SERVO_STALL_NM went 2.94 -> 4.50 in b85a100, which was an accident: that commit
is about cell holders and swept up an edit made minutes earlier in another
session.  Worse, it left HEAD internally inconsistent - mini_dog.py at 4.50 with
ros2/'s urdf still emitting effort="2.94".  This commit regenerates and closes
that; the constant itself is not re-committed here because it is already in.

Steps 4, 5 and 6 in full:

* FEA.  `stall` is the fourth case and scales directly with the constant, so
  every stall SF moved by exactly 1.53x and nothing else moved.  On --orient's
  build-direction index: shin_A 19.36 -> 12.65, hip_bracket_A 8.52 -> 5.57,
  thigh_A 3.08 -> 2.01, cradle_front 1.35 UNCHANGED (governed by land3g, not
  stall, and still the weakest printed part).  Nothing goes below 1.  The crude
  SF column reads thigh_A at 0.8 and that is the worst-orientation figure, not a
  part that fails - the same caveat CLAUDE.md already carries for cradle_front.
* export_sim.py --check: same 2.493 kg, 187 mm stand height, camera axis.
* Step 6 with a control beside it, differing in this one constant and nothing
  else.  Control reproduces the recorded flat baseline to the millimetre.
  flat 482.8 -> 506.3 mm; terrain 350.8 -> 364.3; course 1/7 corridor 1634 ->
  3/7 corridor 2174.  Every arm goes up and that is the model getting stronger,
  not the robot getting better: (forcerange - frictionloss)/damping goes
  2.01 -> 3.15 rad/s, past the ~1.8 the bench measured under the 1 kg arm.

Also resolves PLAN.md's training blocker #2 in rl/'s favour - rl/'s emergent
k_u*12 = 4.23 was within 6 % of the truth and ros2/'s datasheet 2.94 was not.

Two new bench tools, both with selftests.  torque_limit.py writes TORQUE_LIMIT
and reads it back, and refuses while torque is enabled; register 48 is SRAM and
reloads from MAX_TORQUE on every power-up, so it has to be re-applied every
session and after every supply change.  torque_hold.py is a long steady push
with a per-second current profile.

DO NOT READ A SCALE OFF sweep.py --traj stall.  Its 0.8 s bursts are right for
the electrical fit and wrong for an instrument: arm inertia plus the scale's own
filter ringing add a roughly CONSTANT ~130 g (920 g in bursts against 780 held
at the same rung), so it corrupts the slope as well as the level.  The eleven
burst csvs here are kept for their telemetry and are unusable for force; the
four under superseded-unstable-scale/ were taken while the scale was rocking on
the 33 mm jaw.  Method, the thermal decay (4-7 % in 8 s, the winding warming and
R rising at fixed duty), and three fixture faults that each produced a convincing
wrong answer are written up in robot/README.md, "The stall torque, in
newton-metres".

Co-Authored-By: Claude Opus 5 <noreply@anthropic.com>

File: ros2/smalldog_description/urdf/smalldog.urdf (robot description, URDF)
Before this commit: robot smalldog, 17 links, 16 joints
Joints:
- joint fl_knee: limit lower=-1.8500 upper=1.8500 effort=2.94 velocity=4.71 -> lower=-1.8500 upper=1.8500 effort=4.5 velocity=4.71
- joint fl_pitch: limit lower=-1.3000 upper=1.3000 effort=2.94 velocity=4.71 -> lower=-1.3000 upper=1.3000 effort=4.5 velocity=4.71
- joint fl_roll: limit lower=-0.9000 upper=0.9000 effort=2.94 velocity=4.71 -> lower=-0.9000 upper=0.9000 effort=4.5 velocity=4.71
- joint fr_knee: limit lower=-1.8500 upper=1.8500 effort=2.94 velocity=4.71 -> lower=-1.8500 upper=1.8500 effort=4.5 velocity=4.71
- joint fr_pitch: limit lower=-1.3000 upper=1.3000 effort=2.94 velocity=4.71 -> lower=-1.3000 upper=1.3000 effort=4.5 velocity=4.71
- joint fr_roll: limit lower=-0.9000 upper=0.9000 effort=2.94 velocity=4.71 -> lower=-0.9000 upper=0.9000 effort=4.5 velocity=4.71
- joint rl_knee: limit lower=-1.8500 upper=1.8500 effort=2.94 velocity=4.71 -> lower=-1.8500 upper=1.8500 effort=4.5 velocity=4.71
- joint rl_pitch: limit lower=-1.3000 upper=1.3000 effort=2.94 velocity=4.71 -> lower=-1.3000 upper=1.3000 effort=4.5 velocity=4.71
- joint rl_roll: limit lower=-0.9000 upper=0.9000 effort=2.94 velocity=4.71 -> lower=-0.9000 upper=0.9000 effort=4.5 velocity=4.71
- joint rr_knee: limit lower=-1.8500 upper=1.8500 effort=2.94 velocity=4.71 -> lower=-1.8500 upper=1.8500 effort=4.5 velocity=4.71
- joint rr_pitch: limit lower=-1.3000 upper=1.3000 effort=2.94 velocity=4.71 -> lower=-1.3000 upper=1.3000 effort=4.5 velocity=4.71
- joint rr_roll: limit lower=-0.9000 upper=0.9000 effort=2.94 velocity=4.71 -> lower=-0.9000 upper=0.9000 effort=4.5 velocity=4.71

Commit message: bench: the no-load speed is 3.86 rad/s, and it is a plateau (step 3c)
Measured on the stand with the hub free: 3.864 rad/s from the position, 3.835
from PRESENT_SPEED, 12.1 V.  The vendor's 4.71 was 22 % high, and it was the
last vendor number in the speed chain.  SERVO_NOLOAD_RADS is 3.86 now, so
joint_velocity_limit, the URDF velocity and rl/'s joint_vel penalty follow it.
The register's speed LSB is verified as a side effect (1-5 %).

The ladder is the finding.  TORQUE_LIMIT 800 and 1000 read the same speed, with
the register flat at 2500 counts/s, while 400 and 600 are linear through the
origin at k_e = 2.32 V*s/rad.  The duty stops mattering around cap 740.  Whether
that is the position loop's profile (A: stall 4.50 stands, the rl law needs a
goal rate cap) or its PWM ceiling (B: the 2.2x stall extrapolation from rungs
200/350/450 is nearer 3.3) is open.  noload_speed.py --pwm - MODE 2, open loop,
same rungs - decides it; written after the adapter came out, not yet run.

The tool had two defects on its first outing: --min-cap's 900 default filtered
the ladder's own rungs so --duty-ladder ran one, and the fit put a line through
the two plateau points (k_e 3.92, intercept +1.08).  The guard now applies to
the top rung only, and the fit finds the plateau and fits below it.

Ritual: fea.py does not read this constant, so step 4 cannot move and was not
run.  export_sim --check: 2.493 kg, 187 mm, 4 feet down, camera axis right.
The three ros2 sims are bit-identical to the 2026-09-11 rate-limit baseline
(457.8 / 328.8 mm, course 2/7 at 1747): the gait limits against the 3.15
ceiling, which is under 3.86, and the generator now takes min() of the two.
rl/checks/check_model.py 0 FAIL; its stale 2.94/4.71 copies are 4.50/3.86.

Co-Authored-By: Claude Opus 5 (1M context) <noreply@anthropic.com>

File: ros2/smalldog_description/urdf/smalldog.urdf (robot description, URDF)
Before this commit: robot smalldog, 17 links, 16 joints
Joints:
- joint fl_knee: limit lower=-1.8500 upper=1.8500 effort=4.5 velocity=4.71 -> lower=-1.8500 upper=1.8500 effort=4.5 velocity=3.86
- joint fl_pitch: limit lower=-1.3000 upper=1.3000 effort=4.5 velocity=4.71 -> lower=-1.3000 upper=1.3000 effort=4.5 velocity=3.86
- joint fl_roll: limit lower=-0.9000 upper=0.9000 effort=4.5 velocity=4.71 -> lower=-0.9000 upper=0.9000 effort=4.5 velocity=3.86
- joint fr_knee: limit lower=-1.8500 upper=1.8500 effort=4.5 velocity=4.71 -> lower=-1.8500 upper=1.8500 effort=4.5 velocity=3.86
- joint fr_pitch: limit lower=-1.3000 upper=1.3000 effort=4.5 velocity=4.71 -> lower=-1.3000 upper=1.3000 effort=4.5 velocity=3.86
- joint fr_roll: limit lower=-0.9000 upper=0.9000 effort=4.5 velocity=4.71 -> lower=-0.9000 upper=0.9000 effort=4.5 velocity=3.86
- joint rl_knee: limit lower=-1.8500 upper=1.8500 effort=4.5 velocity=4.71 -> lower=-1.8500 upper=1.8500 effort=4.5 velocity=3.86
- joint rl_pitch: limit lower=-1.3000 upper=1.3000 effort=4.5 velocity=4.71 -> lower=-1.3000 upper=1.3000 effort=4.5 velocity=3.86
- joint rl_roll: limit lower=-0.9000 upper=0.9000 effort=4.5 velocity=4.71 -> lower=-0.9000 upper=0.9000 effort=4.5 velocity=3.86
- joint rr_knee: limit lower=-1.8500 upper=1.8500 effort=4.5 velocity=4.71 -> lower=-1.8500 upper=1.8500 effort=4.5 velocity=3.86
- joint rr_pitch: limit lower=-1.3000 upper=1.3000 effort=4.5 velocity=4.71 -> lower=-1.3000 upper=1.3000 effort=4.5 velocity=3.86
- joint rr_roll: limit lower=-0.9000 upper=0.9000 effort=4.5 velocity=4.71 -> lower=-0.9000 upper=0.9000 effort=4.5 velocity=3.86
