Commit message: ros2: the joint limits now come from the ROM scan, and the sim settled with straight legs
A read-only review of ros2/ found the generator hand-typing the one number
everything downstream derives its limits from. J_LIM = {0.90, 1.30, 1.85}
was commented "from the CAD ROM scan"; the scan says +-90/+-90/+-110 deg and
3d/export_sim.py reads it, so the two exporters shipped robots with different
mechanical limits and rl/ trained against the narrower one. The generator now
reads the scan through export_sim.joint_rom()/limits(), carries the signed
per-leg pairs through joints_of(), the URDF and the MJCF, emits them as
joint_limits_rad_signed beside the per-kind values, and asserts symmetry so
nobody is silently clipped if the scan ever becomes asymmetric. Soft limits
0.78/1.18/1.73 -> 1.45/1.45/1.80 rad. The decision to widen was the user's;
it reaches rl/ (retrain, recorded in rl/CLAUDE.md) and the real robot's
runtime clamp (one paragraph added to robot/README.md, where the encoder-wrap
problem in bring-up step 3 is now +-946 counts of roll where it was +-508).

standalone_sim.settle() called joint_targets once with dt = 0, so the rate
limiter emitted 3e-4 rad and the robot "settled" at q ~ 0 - straight legs,
199 mm - and the hold 1s drop was the gait ramping to stance. It seeds the
limiter from the stance now. Clocking the gait every settle step instead was
tried and rejected: standing satisfies _ground()'s landing test, each leg
latches a _gz offset, and the robot flips on terrain inside 5 s.

Step 6 re-baseline, same tree, same seeds - before / settle only / after
(settle + CAD limits): flat 457.8 / 457.9 / 457.9 mm; terrain seeds 7..12
347 +-18 / 420 +-16 / 419 +-16 mm, 0/6 down throughout; course seeds 7/8/9
2-7 1747, 1-7 1597, 2-7 1812 all upright / 0-7 731 DOWN, 2-7 1873, 2-7 1911 /
1-7 1663, 2-7 1733, 2-7 1836 all upright. Course seed 7 is a coin across the
2x2 and is reported as such in 3d/CLAUDE.md. rl/checks/check_model.py 0 FAIL;
smalldog_walker 11 passed; robot/runtime/calib.py --selftest passes on the new
robot_params.json unchanged.

Also in the generator: SCENE's offwidth/offheight were 1400x1000 literals
while the camera's resolution is md.CAM_PIX = 3840x2160, so the offscreen
buffer was smaller than the image read out of it (derived now, and the C++
refuses the mismatch); the URDF shin collision cylinder was synthesised from
pos while the MJCF used fromto, 2.5 mm apart (one source now).

Elsewhere: foot_contact.py's pad/tripod arms forced condim 3 against a
condim-4 control and every label still said 3; keyboard_teleop busy-looped
on stdin EOF ('' in 'rf' is True) and disagreed with standalone_sim and the
README on the body-height band (one band now); walker.launch.py spawned the
walker without use_sim_time or imu_topic; view_robot.launch.py and the rviz2
dep contradicted the README's own rule; three exec_depends the launch file
needs were undeclared; nv printed as dof; README's LiDAR figures were the
catalogue 10 Hz / 2160 points against the measured 12 Hz / ~5200, the test
count 7 against 11, and the bare pytest command cannot run in this pixi env
without PYTEST_DISABLE_PLUGIN_AUTOLOAD=1.

The mujoco_ros2_control submodule moves to 4d92aa8: the dead PID block and
its advertised gains, effort from qfrc_actuator, guarded actuator ids, a
bool init(), and a camera-vs-buffer check. Built clean with colcon.

Co-Authored-By: Claude Fable 5.1 <noreply@anthropic.com>

File: ros2/smalldog_description/urdf/smalldog.urdf (robot description, URDF)
Before this commit: robot smalldog, 17 links, 16 joints
Joints:
- joint fl_knee: limit lower=-1.8500 upper=1.8500 effort=4.5 velocity=3.86 -> lower=-1.9199 upper=1.9199 effort=4.5 velocity=3.86
- joint fl_pitch: limit lower=-1.3000 upper=1.3000 effort=4.5 velocity=3.86 -> lower=-1.5708 upper=1.5708 effort=4.5 velocity=3.86
- joint fl_roll: limit lower=-0.9000 upper=0.9000 effort=4.5 velocity=3.86 -> lower=-1.5708 upper=1.5708 effort=4.5 velocity=3.86
- joint fr_knee: limit lower=-1.8500 upper=1.8500 effort=4.5 velocity=3.86 -> lower=-1.9199 upper=1.9199 effort=4.5 velocity=3.86
- joint fr_pitch: limit lower=-1.3000 upper=1.3000 effort=4.5 velocity=3.86 -> lower=-1.5708 upper=1.5708 effort=4.5 velocity=3.86
- joint fr_roll: limit lower=-0.9000 upper=0.9000 effort=4.5 velocity=3.86 -> lower=-1.5708 upper=1.5708 effort=4.5 velocity=3.86
- joint rl_knee: limit lower=-1.8500 upper=1.8500 effort=4.5 velocity=3.86 -> lower=-1.9199 upper=1.9199 effort=4.5 velocity=3.86
- joint rl_pitch: limit lower=-1.3000 upper=1.3000 effort=4.5 velocity=3.86 -> lower=-1.5708 upper=1.5708 effort=4.5 velocity=3.86
- joint rl_roll: limit lower=-0.9000 upper=0.9000 effort=4.5 velocity=3.86 -> lower=-1.5708 upper=1.5708 effort=4.5 velocity=3.86
- joint rr_knee: limit lower=-1.8500 upper=1.8500 effort=4.5 velocity=3.86 -> lower=-1.9199 upper=1.9199 effort=4.5 velocity=3.86
- joint rr_pitch: limit lower=-1.3000 upper=1.3000 effort=4.5 velocity=3.86 -> lower=-1.5708 upper=1.5708 effort=4.5 velocity=3.86
- joint rr_roll: limit lower=-0.9000 upper=0.9000 effort=4.5 velocity=3.86 -> lower=-1.5708 upper=1.5708 effort=4.5 velocity=3.86

File: ros2/smalldog_ros_control/description/urdf/smalldog-mujoco.urdf.xacro (robot description, xacro)
@@ -7,11 +7,14 @@
       <plugin>mujoco_ros2_control/MujocoSystem</plugin>
     </hardware>
-    <xacro:macro name="pid_joint" params="name">
+    <!-- No PID gains here, and no "_pid" command interface.  They were never used:
+         MujocoSystem::write() writes the position command straight to the MuJoCo position
+         actuator, and the two control_toolbox::Pid it built out of position_kp/ki/kd/i_max
+         were constructed and never called - so turning these knobs did nothing at all.
+         The real gains are the actuator's own kp/dampratio in the MJCF, which come from
+         mini_dog.py's MJ_KP / MJ_DAMPRATIO (measured on the bench, 2026-09-09).
+         Removed 2026-09-11 together with the dead branch in the plugin. -->
+    <xacro:macro name="mj_joint" params="name">
       <joint name="${name}">
-        <param name="position_kp">120</param>
-        <param name="position_ki">0</param>
-        <param name="position_kd">3</param>
-        <param name="position_i_max">10</param>
-        <command_interface name="position_pid"/>
+        <command_interface name="position"/>
         <state_interface name="position">
           <param name="initial_value">0</param>
@@ -21,16 +24,16 @@
       </joint>
     </xacro:macro>
-   <xacro:pid_joint name="fl_roll" />
-   <xacro:pid_joint name="fl_pitch" />
-   <xacro:pid_joint name="fl_knee" />
-   <xacro:pid_joint name="fr_roll" />
-   <xacro:pid_joint name="fr_pitch" />
-   <xacro:pid_joint name="fr_knee" />
-   <xacro:pid_joint name="rl_roll" />
-   <xacro:pid_joint name="rl_pitch" />
-   <xacro:pid_joint name="rl_knee" />
-   <xacro:pid_joint name="rr_roll" />
-   <xacro:pid_joint name="rr_pitch" />
-   <xacro:pid_joint name="rr_knee" />
+   <xacro:mj_joint name="fl_roll" />
+   <xacro:mj_joint name="fl_pitch" />
+   <xacro:mj_joint name="fl_knee" />
+   <xacro:mj_joint name="fr_roll" />
+   <xacro:mj_joint name="fr_pitch" />
+   <xacro:mj_joint name="fr_knee" />
+   <xacro:mj_joint name="rl_roll" />
+   <xacro:mj_joint name="rl_pitch" />
+   <xacro:mj_joint name="rl_knee" />
+   <xacro:mj_joint name="rr_roll" />
+   <xacro:mj_joint name="rr_pitch" />
+   <xacro:mj_joint name="rr_knee" />
     <!-- Body IMU.  mujoco_ros2_control keys off the name: it strips everything after the
          last underscore and looks for MuJoCo sensors <prefix>_quat / _gyro / _accel, and

Commit message: 3d: the three CAD defects the review recorded, and PART_SOLIDS is back to one row
MAC.md recorded three geometry defects on 2026-09-11 rather than fixing them
in the pass that found them. All three are fixed here, and every step of the
ladder was run against the final tree.

- The GPS mast's feet were a literal (-52, +-38) while DECK_SCREWS had moved
  the rear pair to |y| = 41: the mount's M3_CLR holes and the deck's were
  3 mm apart. GPS_X/GPS_Y are derived from DECK_SCREWS[0] now, so the mast
  follows the deck by construction. The pad could not simply move - clipped
  to the lip face it left 0.05 mm of wall round an M3 hole - so the head
  relief chassis_top already cuts in the lip at every screw goes full depth at
  that pair and runs to the deck's end (DECK_LIP_*). Pad-vs-deck 70.2 -> 0 mm3.
- camera_mount's front retaining wall came off as two loose bodies (529 and
  105 mm3) because the board pocket ran the full length of the part. The
  pocket stops CLR short of the board's far end (2.06 mm of end wall, which
  is also the board's stop in y), and a CAM_CAP = 1.2 mm roof bridges the
  channel over the board from the lens relief to the board's near end. Three
  solids -> one, 3657 mm3; lifting the module now meets 2.5..22 mm3 of plastic
  where the old part met none. Neither camera screw moves.
- The Orange Pi's rear standoff pair floated 0.2 mm past the deck's end (two
  384 mm3 orphans). A local tab (OPI_TAB_*) carries them, guarded by
  OPI_TAB_X < -BODY_L/2 so a measured hole pattern deletes it without an edit;
  the pattern keeps its verify marker. Moving OPI_X instead would have put
  OPI_BOX into the LiDAR pedestal.

PART_SOLIDS is {servo_gauge: 2} - two of its three rows were defects it was
permitting rather than describing, and 3d/CLAUDE.md now says so.

+0.79 g of plastic, robot 2.4932 -> 2.4940 kg. ROM unmoved, every clear: line
green, export_sim --check 4 feet down / upright +1.00 / 187 mm. FEA: not one
inter-layer SF moved (three in-plane stand4 figures by 0.1 at SF ~100). Sim,
control / +0.79 g dead mass on the unchanged tree / after: flat 457.9 / - /
457.9; terrain seeds 7..12 419 +-16 0/6 down / 393 +-29 1/6 / 403 +-34 1/6;
course 1-7 1663, 2-7 1733, 2-7 1836 / 1-7 1654, 0-7 449 down, 2-7 1838 /
2-7 1791, 0-7 451 down, 2-7 1842. Seed 8 falls in the dead-mass arm and the
changed arm at the same distance to 2 mm - the documented mass cliff, not the
geometry. No step-6 re-baseline.

Co-Authored-By: Claude Fable 5.1 <noreply@anthropic.com>

File: ros2/smalldog_description/urdf/smalldog.urdf (robot description, URDF)
Before this commit: robot smalldog, 17 links, 16 joints
Links:
- link base_link: mass 1.55858 -> 1.55937

Commit message: 3d: SERVO_STALL_NM 4.50 → 3.2, the measured full-duty peak, and MJ_DAMPING into the same calibration
The rig at full duty read 3.2 N·m cold at 12 V (0.40 N·m/V of drive to ~5.5 V, ~0.20
above); 4.50 was the low-duty line extrapolated past its last rung. It feeds FEA's stall
column (inter-layer SF 1.6/0.8/3.2/1.9 → 2.2/1.1/4.5/2.7) and both sims' forcerange.

MJ_DAMPING 1.37 → 0.92: the ladder's total is in its own calibration (k_t 0.596 N·m/V,
before the gearbox's load loss), the stall in the scale's (0.400, after it), and the joint
ceiling divides one by the other. One calibration: 1.37 × 0.400/0.596. Ceiling 3.15 →
3.28 rad/s; walk.py's fitted gait moves to 0.11 m/s at 1.35 s. rl/ zeroes MJ_DAMPING.

Ladder, six steps: no !!, probes unchanged, export --check upright, step 6 flat 522.8
(control with 4.50/1.37 on the same mesh 456.7), terrain seeds 7…12 415 ±44 mm 0/6
down (was 403 ±34, 1/6), course 7/8/9 1986/1716/2149 all upright (was 1791/451 down/1842).
check_model.py 0 FAIL; its forcerange copy now WARNs on divergence instead of INFO.

The held ~2.3 N·m and the 2 s protection timer are not a sim constant — a per-joint
budget for runtime/safety.py, PLAN.md 3d, open.

Co-Authored-By: Claude Opus 5 (1M context) <noreply@anthropic.com>

File: ros2/smalldog_description/urdf/smalldog.urdf (robot description, URDF)
Before this commit: robot smalldog, 17 links, 16 joints
Links:
- link base_link: mass 1.55937 -> 1.55900
Joints:
- joint fl_knee: limit lower=-1.9199 upper=1.9199 effort=4.5 velocity=3.86 -> lower=-1.9199 upper=1.9199 effort=3.2 velocity=3.86
- joint fl_pitch: limit lower=-1.5708 upper=1.5708 effort=4.5 velocity=3.86 -> lower=-1.5708 upper=1.5708 effort=3.2 velocity=3.86
- joint fl_roll: limit lower=-1.5708 upper=1.5708 effort=4.5 velocity=3.86 -> lower=-1.5708 upper=1.5708 effort=3.2 velocity=3.86
- joint fr_knee: limit lower=-1.9199 upper=1.9199 effort=4.5 velocity=3.86 -> lower=-1.9199 upper=1.9199 effort=3.2 velocity=3.86
- joint fr_pitch: limit lower=-1.5708 upper=1.5708 effort=4.5 velocity=3.86 -> lower=-1.5708 upper=1.5708 effort=3.2 velocity=3.86
- joint fr_roll: limit lower=-1.5708 upper=1.5708 effort=4.5 velocity=3.86 -> lower=-1.5708 upper=1.5708 effort=3.2 velocity=3.86
- joint rl_knee: limit lower=-1.9199 upper=1.9199 effort=4.5 velocity=3.86 -> lower=-1.9199 upper=1.9199 effort=3.2 velocity=3.86
- joint rl_pitch: limit lower=-1.5708 upper=1.5708 effort=4.5 velocity=3.86 -> lower=-1.5708 upper=1.5708 effort=3.2 velocity=3.86
- joint rl_roll: limit lower=-1.5708 upper=1.5708 effort=4.5 velocity=3.86 -> lower=-1.5708 upper=1.5708 effort=3.2 velocity=3.86
- joint rr_knee: limit lower=-1.9199 upper=1.9199 effort=4.5 velocity=3.86 -> lower=-1.9199 upper=1.9199 effort=3.2 velocity=3.86
- joint rr_pitch: limit lower=-1.5708 upper=1.5708 effort=4.5 velocity=3.86 -> lower=-1.5708 upper=1.5708 effort=3.2 velocity=3.86
- joint rr_roll: limit lower=-1.5708 upper=1.5708 effort=4.5 velocity=3.86 -> lower=-1.5708 upper=1.5708 effort=3.2 velocity=3.86

Commit message: 3d: the L2 on a nose bracket, axis forward (LIDAR_TILT 45 -> 90)
lidar_mount is a bracket now: the old base plate and deck interface untouched (four
bolts, camera-tab pockets, the flat at 63.5), a 4 mm stem up the chassis front face,
two ribs between the L2's screw heads, a @64 x 7 seat disc recessed to 4.5 behind.
40.0 g against the seat's 38.5. LIDAR_SEAT_Z = 95 is set by the camera: the L2 hangs
65 mm out over the lens and its underside has to stay out of the face band -
camera_clear() now charges the L2 envelope (lidar_module()) every build, and the L2 is
in interference() and the hip-roll scan. Both exporters build its inertia from
lidar_box_xyz(). lidar_seat_min() is gone with the tilted seat.

export_sim --check: the floor from +4 mm past the leading foot (was +226), 2277
returns/frame (was 819). FEA identical. Flat trot 543.8 (control 524.8); terrain
7..12: 458 +-30, 2/6 down (11, 12) against 0/6 - the +1.5 g control drops 12 too;
course 7/8/9: 2225 / 2153 / 2266, all upright. Base-link CoM +4.9 mm forward.

Co-Authored-By: Claude Opus 5 (1M context) <noreply@anthropic.com>

File: ros2/smalldog_description/urdf/smalldog.urdf (robot description, URDF)
Before this commit: robot smalldog, 17 links, 16 joints
Links:
- link base_link: mass 1.56048 -> 1.56203
Joints:
- joint lidar_link_joint: origin xyz=0.0734663 0 0.0914663 rpy=0 0.785398 0 -> xyz=0.1075 0 0.095 rpy=0 1.5708 0

Commit message: 3d: cable routes - bus and low windows in both end walls, tie slots on the driven arms, a WAGO power node in the rear strip
The front cradle frame was a sealed box with the two front roll servos' ports
inside it: the bus window was cut in the rear wall only. Both end walls now
have it, plus a 14 x 6 low window on the floor for the pitch and knee leads
coming back under the cradle rail on the centreline. Each lead crosses one
joint, on the driven arm's outer face through the axis; fork() cuts two tie
slots there, 16 and 20 mm out on the link side, where the arm is the spine web
and not the disc with the hub screws in it. The shin's fork gets none.

The power node is two WAGO 221-415 lever nuts, P+ and P-, glued on the rear
upper cradle-screw seats with the levers toward the centreline (NODE_*,
node_clear() every build). The strip is 17.6 mm deep and 14.8 behind the seats
against a 221's 18.6 along the wire, so one pair is all it holds: pack lead and
four legs. The charge branch and the buck feed take the MIDI holder's stud
instead. The ESP32/URT-1 rib that split the strip is gone.

One 18 AWG pair per leg replaces power through *1's connector (POWER.md).

Mass -1.3 g. FEA within noise (hip_bracket_A --orient 7.83 -> 7.79, thigh_A
2.83 -> 2.82). Flat trot 542.4 against a -1.3 g control of 537.4; terrain and
course move with the gram, not the geometry - the control is in 3d/CLAUDE.md.

Co-Authored-By: Claude Opus 5 (1M context) <noreply@anthropic.com>

File: ros2/smalldog_description/urdf/smalldog.urdf (robot description, URDF)
Before this commit: robot smalldog, 17 links, 16 joints
Links:
- link base_link: mass 1.56203 -> 1.56092
- link fl_hip: mass 0.09016 -> 0.09005
- link fl_thigh: mass 0.09707 -> 0.09697
- link fr_hip: mass 0.09016 -> 0.09005
- link fr_thigh: mass 0.09707 -> 0.09697
- link rl_hip: mass 0.09016 -> 0.09005
- link rl_thigh: mass 0.09707 -> 0.09697
- link rr_hip: mass 0.09016 -> 0.09005
- link rr_thigh: mass 0.09707 -> 0.09697

Commit message: 3d: the end-wall windows are cut through the wall, and panel_clear() checks that they are
The cut box in chassis_bottom() sat outside the wall - the sign of the wall-
thickness term was inverted - so the rear bus window vanished (a zero-size box)
and the front one stopped 1.8 mm short. panel_clear() looks outward from the
wall for a plug's room and passed both. It now also intersects each window's
own box, through the wall, with the tray; the XT30 pocket is excluded because
its lip is the point.

-3.5 g. The step-6 control at the same mass on the previous geometry is in
3d/CLAUDE.md: seeds 9 and 10 go down with the windows and stand without, on a
metric chaotic in the gram - 4/6 against 2/6 at n = 6.

Co-Authored-By: Claude Opus 5 (1M context) <noreply@anthropic.com>

File: ros2/smalldog_description/urdf/smalldog.urdf (robot description, URDF)
Before this commit: robot smalldog, 17 links, 16 joints
Links:
- link base_link: mass 1.56092 -> 1.55906

Commit message: 3d: the Orange Pi 5 Pro measured and cased, the IMU inside the case
The board off the vendor drawing (ref/opi/: 89.1 x 56, holes 58 x 49, column 7.6 mm
from the micro-SD end) in its bought 105 x 70.5 x 40 case, micro-SD end forward at
OPI_X = -33 on four 6.5 mm spacer bosses, bolted from under the deck with M2.5 x 17
into the case's own spacers (heads flush in counterbores - the battery lid is 0.6 mm
below). ELECTRONICS_KG 195 -> 250 g measured. The GPS mast's knee, both numbers, now
derives from OPI_BOX: seat 65 -> 95.7. The deck tab and the nut slots are gone.

The IMU moves into the case: taped face up on the bottom plate at (0, +15, 40.4), in the
strip beside the M.2 module, wired to the Pi's underside I2C pads; both exporters read
the mass box from imu_box() and the site from imu_xyz(). The deck's two IMU standoffs
and their formed threads are gone. Moving the site is an RL re-baseline.

New probes: opi_clear() (case vs the LiDAR bracket, rear feet vs the deck's end),
opi_bolt_engage(), and imu_clear() against the M.2 band, the case spacers and the PCB.
All six steps green; FEA ground columns down ~2 % with the mass; flat trot 526.0.

Still **verify**: OPI_CASE_PCB (where the board sits in the case), the case's spacer
gap and radius, the bolt against the spacer's thread depth.

Co-Authored-By: Claude Opus 5 (1M context) <noreply@anthropic.com>

File: ros2/smalldog_description/urdf/smalldog.urdf (robot description, URDF)
Before this commit: robot smalldog, 17 links, 16 joints
Links:
- link base_link: mass 1.55906 -> 1.61547
Joints:
- joint gps_joint: origin xyz=-0.05200 0.00000 0.07260 rpy=0 0 0 -> xyz=-0.05200 0.00000 0.10330 rpy=0 0 0

Commit message: 3d: the buck rides on the Pi's case top under the GPS platform; Pi bolts M2.5 x 11 flat heads; the bench test pack
BUCK_* / buck_clear() / buck_com(): the XL4015 on foam tape on the Orange Pi's case
top, the one 17 mm of air on the robot (rear strip 14.05, side strips 8.4); its 18 g
out of ELECTRONICS_KG's allowance, GPS_LAND derives from its top plus BUCK_AIR (seat
95.7 -> 96.6). OPI_BOLT_L 17 -> 11, hex-socket flat heads seated up inside the spacer
bosses (OPI_SEAT_D, opi_bolt_check()), 2.5 mm into the case's brass spacers. Baseline
flat trot 537.3 mm, description regenerated. test_pack.py: the screw-terminal 3S1P
18650 holder for the bench, not a robot part. ref/imu: where the IMU sits in the case,
with the photo; ref/power: the buck trimmed to 5.0 V under load.

Co-Authored-By: Claude Opus 5 (1M context) <noreply@anthropic.com>

File: ros2/smalldog_description/urdf/smalldog.urdf (robot description, URDF)
Before this commit: robot smalldog, 17 links, 16 joints
Links:
- link base_link: mass 1.61547 -> 1.61539
Joints:
- joint gps_joint: origin xyz=-0.05200 0.00000 0.10330 rpy=0 0 0 -> xyz=-0.05200 0.00000 0.10420 rpy=0 0 0

Commit message: straight_test: 40 s for a parked head (~25 s measured)
Co-Authored-By: Claude Opus 5 (1M context) <noreply@anthropic.com>

File: ros2/smalldog_description/urdf/smalldog.urdf (robot description, URDF)
Before this commit: robot smalldog, 17 links, 16 joints
Links:
- link base_link: mass 1.61539 -> 1.61533
